File: Main_H743VI.kicad_pcb (KiCad board)
At the start: 4 copper layers, 150 x 100 mm, 75 parts, among them J1 ST-LINK, J10 AS7265X, J11 TFT_FMC, J12 SERVO1, J13 USER_GPIO, J14 TFT_SPI, J15 SERVO2, J16 FAN, J17 ADC_IN, J18 BME280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

Commit message: snapshotprior to autorout
Parts:
- moved R18 0.83 mm to (198.8, 41.3)
- turned D3 to 180 degrees
- turned L1 to -90 degrees
Routing:
- net VCC: track 0.00 -> 27.6 mm
- net Net-(U2-BOOST): track 0.00 -> 22.4 mm
- net Net-(D3-K): track 0.00 -> 19.7 mm
- net GND: track 0.00 -> 12.4 mm, vias 0 -> 2
- net +12V: track 0.00 -> 5.02 mm, vias 0 -> 2

Commit message: end of day snapshot
Parts:
- moved R7 56.6 mm to (94.8, 42.9)
- moved J7 56.6 mm to (81.5, 45.7)
- moved J18 56.6 mm to (89.2, 45.9)
- moved R8 56.6 mm to (94.8, 38.5)
- moved J6 42.0 mm to (82.6, 81.0)
- moved J17 29.3 mm to (97.4, 66.2), turned to 0 degrees
- moved D1 16.8 mm to (133.4, 98.2)
- moved R5 16.8 mm to (133.4, 93.8)
- moved J10 16.5 mm to (82.1, 65.2)
- moved R10 16.5 mm to (88.8, 57.6)
- moved R9 16.5 mm to (88.7, 62.2)
- moved R18 15.2 mm to (184.2, 45.9)
- moved C1 10.3 mm to (117.4, 28.0), turned to 90 degrees
- moved R20 10.1 mm to (147.1, 30.7)
- moved J2 10.00 mm to (147.1, 25.6), turned to -90 degrees
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Routing:
- net +12V: track 5.02 -> 2.48 mm, vias 2 -> 0
- net GND: track 12.4 -> 10.3 mm, vias 2 -> 0
